File: iolite.kicad_pcb (KiCad board)
At the start: 2 copper layers, 149 x 100 mm, 51 parts, among them IC1 ATMEGA168-P, J2 DB9, P1 CONN_CTL_DATA, P2 CONN_ADDR, P3 SLOT_PWR, P4 SLOT1, P5 SLOT2, P6 CONN_01X02, P7 SLOT_EX_ADDR, U1 74LS138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

Commit message: updated schematics
Parts:
- renumbered ISP to ISP1
Connections:
- IC1 pad 17: /~IRQ7~/MOSI -> /~IRQ7
- ISP1 pad 4: /~IRQ7~/MOSI -> /~IRQ7
Routing:
- net /~IRQ7: track 2.48 -> 80.2 mm, vias 0 -> 1
- net /~IRQ7~/MOSI: track 7.40 -> 0.00 mm
- net /~SYS_RESET: track 146.8 -> 148.6 mm
- net VCC: track 620.9 -> 622.3 mm
